Commit message: working on noetic

File: ouster_description/urdf/OS1-64.urdf.xacro (robot description, xacro)
@@ -24,6 +24,5 @@
          <origin xyz="0 0 0.0" rpy="0 0 1.5707" />
          <geometry>
-	         <mesh filename="package://ouster_description/meshes/os1_64.dae" />
-           <!-- <cylinder length="0.073" radius="0.04" /> -->
+	         <mesh filename="package://ouster_description/meshes/os1_64.dae"/>
          </geometry>
       </visual>
@@ -80,18 +79,18 @@
     </gazebo>
     <!-- IMU -->
-  <gazebo>
-    <plugin name="imu_controller" filename="libhector_gazebo_ros_imu.so">
-      <robotNamespace>/</robotNamespace>
-      <updateRate>100.0</updateRate>
-      <bodyName>${imu_link}</bodyName>
-      <topicName>${topic_imu}</topicName>
-      <accelDrift>0.005 0.005 0.005</accelDrift>
-      <accelGaussianNoise>0.005 0.005 0.005</accelGaussianNoise>
-      <rateDrift>0.005 0.005 0.005 </rateDrift>
-      <rateGaussianNoise>0.005 0.005 0.005 </rateGaussianNoise>
-      <headingDrift>0.005</headingDrift>
-      <headingGaussianNoise>0.005</headingGaussianNoise>
-    </plugin>
-  </gazebo>
+    <gazebo>
+      <plugin name="imu_controller" filename="libhector_gazebo_ros_imu.so">
+        <robotNamespace>/</robotNamespace>
+        <updateRate>100.0</updateRate>
+        <bodyName>${imu_link}</bodyName>
+        <topicName>${topic_imu}</topicName>
+        <accelDrift>0.005 0.005 0.005</accelDrift>
+        <accelGaussianNoise>0.005 0.005 0.005</accelGaussianNoise>
+        <rateDrift>0.005 0.005 0.005 </rateDrift>
+        <rateGaussianNoise>0.005 0.005 0.005 </rateGaussianNoise>
+        <headingDrift>0.005</headingDrift>
+        <headingGaussianNoise>0.005</headingGaussianNoise>
+      </plugin>
+    </gazebo>
   </xacro:macro>
 </robot>

File: ouster_description/urdf/example.urdf.xacro (robot description, xacro)
@@ -28,7 +28,7 @@
     </inertial>
   </link>
-  <xacro:include filename="$(find ouster_description)/urdf/OS1-64.urdf.xacro"/>
-  <OS1-64 parent="base_link" name="os1_sensor" hz="10" samples="220">
+  <xacro:include filename="/home/fdcl/Ouster/gazebo_ws_wilselby/src/ouster_example/ouster_description/urdf/OS1-64.urdf.xacro"/>
+  <xacro:OS1-64 parent="base_link" name="os1_sensor" hz="10" samples="220">
     <origin xyz="0 0 1.2" rpy="0 0 0" />
-  </OS1-64>
+  </xacro:OS1-64>
 </robot>

Commit message: ship added. mesh needs fixing

File: ouster_description/urdf/OS1-64.urdf.xacro (robot description, xacro)
@@ -2,7 +2,7 @@
 <robot xmlns:xacro="http://www.ros.org/wiki/xacro" name="OS1-64">
   <xacro:property name="M_PI" value="3.1415926535897931" />
-  <xacro:macro name="OS1-64" params="*origin parent:=base_link name:=os1_sensor topic_points:=/os1_cloud_node/points topic_imu:=/os1_cloud_node/imu hz:=10 lasers:=64 samples:=512 min_range:=0.9 max_range:=75.0 noise:=0.008 min_angle:=-${M_PI} max_angle:=${M_PI} lidar_link:=os1_lidar imu_link:=os1_imu vfov_min:=-.26 vfov_max:=.26">
+  <xacro:macro name="OS1-64" params="*origin parent:=base_link name:=os1_sensor topic_points:=/os1_cloud_node/points topic_imu:=/os1_cloud_node/imu hz:=10 lasers:=32 samples:=512 min_range:=0.5 max_range:=30.0 noise:=0.008 min_angle:=-${M_PI} max_angle:=${M_PI} lidar_link:=os1_lidar imu_link:=os1_imu vfov_min:=-.785 vfov_max:=.785">
     <joint name="${name}_mount_joint" type="fixed">
-      <xacro:insert_block name="origin" />
+      <origin xyz="0 0 0.0" rpy="0 0 0" />
       <parent link="${parent}"/>
       <child link="${name}"/>
@@ -10,20 +10,20 @@
     <link name="${name}">
       <inertial>
-         <mass value="0.33"/>
-         <origin xyz="0 0 0.0365" rpy="0 0 0" />
-         <inertia ixx="0.000241148" ixy="0" ixz="0"
-          iyy="0.000241148" iyz="0" izz="0.000264"/>
+        <mass value="0.33"/>
+        <origin xyz="0 0 0.05" rpy="0 0 0" />
+        <inertia ixx="0.000241148" ixy="0" ixz="0"
+                  iyy="0.000241148" iyz="0" izz="0.000264"/>
       </inertial>
       <collision name="base_collision">
-         <origin xyz="0 0 0.0365" rpy="0 0 0" />
-         <geometry>
- 	        <cylinder radius="0.04" length="0.073"/>
-         </geometry>
+        <origin xyz="0 0 0.05" rpy="0 0 0" />
+        <geometry>
+          <cylinder radius="0.04" length="0.073"/>
+        </geometry>
       </collision>
       <visual name="base_visual">
-         <origin xyz="0 0 0.0" rpy="0 0 1.5707" />
-         <geometry>
-	         <mesh filename="package://ouster_description/meshes/os1_64.dae"/>
-         </geometry>
+        <origin xyz="0 0 0.05" rpy="0 0 1.5707" />
+        <geometry>
+          <mesh filename="package://ouster_description/meshes/os1_64.dae"/>
+        </geometry>
       </visual>
     </link>
@@ -33,5 +33,5 @@
       <parent link="${name}" />
       <child link="${imu_link}" />
-      <origin xyz="0.006253 -0.011775 0.007645" rpy="0 0 0" />
+      <origin xyz="0.006253 -0.011775 0.027645" rpy="0 0 0" />
     </joint>
     <gazebo reference="${imu_link}">

File: ouster_description/urdf/example.urdf.xacro (robot description, xacro)
@@ -3,19 +3,23 @@
   <!-- Base Footprint -->
   <link name="base_footprint" />
+  <!-- Make the robot static -->
+  <gazebo>
+    <static>true</static>
+  </gazebo>
   <!-- Base Link -->
   <joint name="footprint" type="fixed" >
    <parent link="base_footprint" />
     <child link="base_link" />
-    <origin xyz="0 0 0.05" rpy="0 0 0" />
+    <origin xyz="0 0 0.00" rpy="0 0 0" />
   </joint>
   <link name="base_link" >
     <visual>
       <geometry>
-        <box size="0.5 0.5 0.1" />
+        <box size="0.3 0.3 0.03" />
       </geometry>
     </visual>
     <collision>
       <geometry>
-        <box size="0.5 0.5 0.1" />
+        <box size="0.3 0.3 0.03" />
       </geometry>
     </collision>
@@ -23,12 +27,12 @@
       <origin xyz="0 0 0"/>
       <mass value="10"/>
-      <inertia ixx="3.0" ixy="0.0" ixz="0.0"
-               iyy="3.0" iyz="0.0"
-               izz="3.0" />
+      <inertia ixx="1.0" ixy="0.0" ixz="0.0"
+               iyy="1.0" iyz="0.0"
+               izz="1.0" />
     </inertial>
   </link>
-  <xacro:include filename="/home/fdcl/Ouster/gazebo_ws_wilselby/src/ouster_example/ouster_description/urdf/OS1-64.urdf.xacro"/>
+  <xacro:include filename="$(find ouster_description)/urdf/OS1-64.urdf.xacro"/>
   <xacro:OS1-64 parent="base_link" name="os1_sensor" hz="10" samples="220">
-    <origin xyz="0 0 1.2" rpy="0 0 0" />
+    <origin xyz="0 0 0.05" rpy="0 0 0" />
   </xacro:OS1-64>
 </robot>

File: output.urdf (robot description, URDF)
Before this commit: robot os1_example, 5 links, 4 joints
Links:
- link base_link: geometry collision box size=0.3 0.3 0.03; visual box size=0.3 0.3 0.03
- link os1_sensor: geometry collision cylinder length=0.073 radius=0.04; visual mesh filename=package://ouster_description/meshes/os1_64.dae
Joints:
- joint footprint: origin xyz=0 0 0.05 rpy=0 0 0 -> xyz=0 0 0.00 rpy=0 0 0
- joint os1_sensor_mount_joint: origin xyz=0 0 1.2 rpy=0 0 0 -> xyz=0 0 0.0 rpy=0 0 0

Commit message: lidar upside down. improve ship, sample poses

File: ouster_description/urdf/OS1-64.urdf.xacro (robot description, xacro)
@@ -3,6 +3,7 @@
   <xacro:property name="M_PI" value="3.1415926535897931" />
   <xacro:macro name="OS1-64" params="*origin parent:=base_link name:=os1_sensor topic_points:=/os1_cloud_node/points topic_imu:=/os1_cloud_node/imu hz:=10 lasers:=32 samples:=512 min_range:=0.5 max_range:=30.0 noise:=0.008 min_angle:=-${M_PI} max_angle:=${M_PI} lidar_link:=os1_lidar imu_link:=os1_imu vfov_min:=-.785 vfov_max:=.785">
+    <!-- _mount_joint connects to base joint -->
     <joint name="${name}_mount_joint" type="fixed">
-      <origin xyz="0 0 0.0" rpy="0 0 0" />
+      <origin xyz="0 0 0.0" rpy="3.14159 0 0" />
       <parent link="${parent}"/>
       <child link="${name}"/>

Commit message: reading pose+cloud topics and can write poses

File: ouster_description/urdf/OS1-64.urdf.xacro (robot description, xacro)
@@ -5,5 +5,6 @@
     <!-- _mount_joint connects to base joint -->
     <joint name="${name}_mount_joint" type="fixed">
-      <origin xyz="0 0 0.0" rpy="3.14159 0 0" />
+      <!-- <origin xyz="5 0 3" rpy="3.14159 0 0" /> -->
+      <origin xyz="0 0 0" rpy="0 0 0" />
       <parent link="${parent}"/>
       <child link="${name}"/>

File: ouster_description/urdf/example.urdf.xacro (robot description, xacro)
@@ -11,5 +11,6 @@
    <parent link="base_footprint" />
     <child link="base_link" />
-    <origin xyz="0 0 0.00" rpy="0 0 0" />
+    <origin xyz="5 0 3" rpy="0 0 0" />
+    <!-- <origin xyz="0 0 0" rpy="0 0 0" /> -->
   </joint>
   <link name="base_link" >

Commit message: normal distribution for r_c

File: ouster_description/urdf/OS1-64.urdf.xacro (robot description, xacro)
@@ -2,5 +2,5 @@
 <robot xmlns:xacro="http://www.ros.org/wiki/xacro" name="OS1-64">
   <xacro:property name="M_PI" value="3.1415926535897931" />
-  <xacro:macro name="OS1-64" params="*origin parent:=base_link name:=os1_sensor topic_points:=/os1_cloud_node/points topic_imu:=/os1_cloud_node/imu hz:=10 lasers:=32 samples:=512 min_range:=0.5 max_range:=30.0 noise:=0.008 min_angle:=-${M_PI} max_angle:=${M_PI} lidar_link:=os1_lidar imu_link:=os1_imu vfov_min:=-.785 vfov_max:=.785">
+  <xacro:macro name="OS1-64" params="*origin parent:=base_link name:=os1_sensor topic_points:=/os1_cloud_node/points topic_imu:=/os1_cloud_node/imu hz:=10 lasers:=32 samples:=512 min_range:=0.3 max_range:=45.0 noise:=0.008 min_angle:=-${M_PI} max_angle:=${M_PI} lidar_link:=os1_lidar imu_link:=os1_imu vfov_min:=-.785 vfov_max:=.785">
     <!-- _mount_joint connects to base joint -->
     <joint name="${name}_mount_joint" type="fixed">

File: ouster_description/urdf/example.urdf.xacro (robot description, xacro)
@@ -34,5 +34,5 @@
   </link>
   <xacro:include filename="$(find ouster_description)/urdf/OS1-64.urdf.xacro"/>
-  <xacro:OS1-64 parent="base_link" name="os1_sensor" hz="10" samples="220">
+  <xacro:OS1-64 parent="base_link" name="os1_sensor">
     <origin xyz="0 0 0.05" rpy="0 0 0" />
   </xacro:OS1-64>

Commit message: sampling for sim-to-real complete

File: ouster_description/urdf/OS1-64.urdf.xacro (robot description, xacro)
@@ -2,5 +2,5 @@
 <robot xmlns:xacro="http://www.ros.org/wiki/xacro" name="OS1-64">
   <xacro:property name="M_PI" value="3.1415926535897931" />
-  <xacro:macro name="OS1-64" params="*origin parent:=base_link name:=os1_sensor topic_points:=/os1_cloud_node/points topic_imu:=/os1_cloud_node/imu hz:=10 lasers:=32 samples:=512 min_range:=0.3 max_range:=45.0 noise:=0.008 min_angle:=-${M_PI} max_angle:=${M_PI} lidar_link:=os1_lidar imu_link:=os1_imu vfov_min:=-.785 vfov_max:=.785">
+  <xacro:macro name="OS1-64" params="*origin parent:=base_link name:=os1_sensor topic_points:=/os1_cloud_node/points topic_imu:=/os1_cloud_node/imu hz:=10 lasers:=32 samples:=512 min_range:=0.3 max_range:=50.0 noise:=0.008 min_angle:=-${M_PI} max_angle:=${M_PI} lidar_link:=os1_lidar imu_link:=os1_imu vfov_min:=-.785 vfov_max:=.785">
     <!-- _mount_joint connects to base joint -->
     <joint name="${name}_mount_joint" type="fixed">

File: ouster_description/urdf/ship.urdf (robot description, URDF)
Before this commit: robot ship_model, 1 links, 0 joints
Links:
- link ship: geometry collision mesh filename=package://ouster_description/meshes/sim-to-real/scaled_Ship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 scale=1 1 1; visual mesh filename=package://ouster_description/meshes/sim-to-real/scaled_Ship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 scale=1 1 1

Commit message: os0-sim beam fixes and new sampling

File: ouster_description/urdf/OS1-64.urdf.xacro (robot description, xacro)
@@ -2,5 +2,5 @@
 <robot xmlns:xacro="http://www.ros.org/wiki/xacro" name="OS1-64">
   <xacro:property name="M_PI" value="3.1415926535897931" />
-  <xacro:macro name="OS1-64" params="*origin parent:=base_link name:=os1_sensor topic_points:=/os1_cloud_node/points topic_imu:=/os1_cloud_node/imu hz:=10 lasers:=32 samples:=512 min_range:=0.3 max_range:=50.0 noise:=0.008 min_angle:=-${M_PI} max_angle:=${M_PI} lidar_link:=os1_lidar imu_link:=os1_imu vfov_min:=-.785 vfov_max:=.785">
+  <xacro:macro name="OS1-64" params="*origin parent:=base_link name:=os1_sensor topic_points:=/os1_cloud_node/points topic_imu:=/os1_cloud_node/imu hz:=10 lasers:=32 samples:=512 min_range:=0.3 max_range:=50.0 noise:=0.02 min_angle:=-${M_PI} max_angle:=${M_PI} lidar_link:=os1_lidar imu_link:=os1_imu vfov_min:=-.80 vfov_max:=.80">
     <!-- _mount_joint connects to base joint -->
     <joint name="${name}_mount_joint" type="fixed">
@@ -77,4 +77,5 @@
             <max_range>${max_range}</max_range>
             <gaussianNoise>${noise}</gaussianNoise>
+            <!-- <beam_intrinsics_path>/home/fdcl/Ouster/gazebo_ws_fdcl/src/ouster_simulation/os0_32_beam_intrinsics.json</beam_intrinsics_path> -->
           </plugin>
         </sensor>
